File: PCB design/ttn-rainfall.sch (KiCad schematic (older format))
At the start: 23 parts

Commit message: Moved files around
Parts:
- Y?: value Crystal -> 16MHz
Changed lines of the file:
@@
 P 6800 2000
 F 0 "Y?" H 6800 2150 50  0000 C CNN
-F 1 "Crystal" H 6800 1850 50  0000 C CNN
+F 1 "16MHz" H 6800 1850 50  0000 C CNN
 F 2 "" H 6800 2000 50  0001 C CNN
 F 3 "" H 6800 2000 50  0001 C CNN

Commit message: PCB drawn
Parts:
- removed C? (x2): 18p, symbol C_Small
- removed Y?: 16MHz, symbol Crystal
- added Q1: CSTCE16M0V53-R0, drawn_by_jpmeijers:RESONATOR_CSTCE16M0V53-R0, symbol RESONATOR_CSTCE16M0V53-R0
- C1, C2, C3, C4, C5, C6: renamed from C?; footprint (none) -> Capacitors_SMD:C_0805
- C9: renamed from C?; value C_Small -> 100n; footprint (none) -> Capacitors_SMD:C_0805
- D1: renamed from D?; footprint (none) -> LEDs:LED_0805
- J1, J3: renamed from J?; footprint (none) -> Pin_Headers:Pin_Header_Straight_1x02_Pitch2.54mm
- J2: renamed from J?; footprint (none) -> Pin_Headers:Pin_Header_Straight_1x01_Pitch2.54mm
- J4: renamed from J?; footprint (none) -> Pin_Headers:Pin_Header_Straight_2x03_Pitch2.54mm
- R1, R2, R3: renamed from R?; footprint (none) -> Resistors_SMD:R_0805
- SW1, SW2: renamed from SW?; footprint (none) -> Buttons_Switches_SMD:SW_SPST_B3SL-1002P
- U1: renamed from U?; footprint (none) -> drawn_by_jpmeijers:RFM95
- U3: renamed from U?; footprint (none) -> TO_SOT_Packages_SMD:TSOT-23_HandSoldering
- gave numbers to parts that had none: 1
Connections:
- net GND: now also Q1.2 (GND)
- net at U2.7 ((PCINT6/XTAL1/TOSC1)PB6): now also Q1.3
- net at U2.8 ((PCINT7/XTAL2/TOSC2)PB7): now also Q1.1
- no-connect marks 5 -> 12
