File: PCB design/ttn-rainfall.kicad_pcb (KiCad board)
At the start: 2 copper layers, 21 parts, among them J1 BATTERY, J2 ANTENNA, J3 UART, J4 ICSP, Q1 CSTCE16M0V53-R0, SW1 SW_Push, SW2 SW_Push, U1 RFM95, U2 ATMEGA328P-AU, U3 TSH251

Commit message: Initial order from allpcb
Other:
- board outline added: 43.2 x 55.9 mm
Changed lines of the file:
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@@
     (area 0 0 0 0)
     (thickness 1.6)
-    (drawings 7)
+    (drawings 15)
     (tracks 455)
     (zones 0)
@@
   (page A4)
   (layers
-    (0 F.Cu signal)
-    (31 B.Cu signal)
+    (0 F.Cu signal hide)
+    (31 B.Cu signal hide)
     (32 B.Adhes user)
     (33 F.Adhes user)
@@
       (net 34 "Net-(Q1-Pad3)"))
   )
+  (gr_line (start 105.41 127) (end 146.05 127) (angle 90) (layer Edge.Cuts) (width 0.15))
+  (gr_line (start 104.14 72.39) (end 104.14 125.73) (angle 90) (layer Edge.Cuts) (width 0.15))
+  (gr_line (start 146.05 71.12) (end 105.41 71.12) (angle 90) (layer Edge.Cuts) (width 0.15))
+  (gr_line (start 147.32 125.73) (end 147.32 72.39) (angle 90) (layer Edge.Cuts) (width 0.15))
+  (gr_arc (start 146.05 125.73) (end 147.32 125.73) (angle 90) (layer Edge.Cuts) (width 0.15))
+  (gr_arc (start 105.41 125.73) (end 105.41 127) (angle 90) (layer Edge.Cuts) (width 0.15))
+  (gr_arc (start 105.41 72.39) (end 104.14 72.39) (angle 90) (layer Edge.Cuts) (width 0.15))
+  (gr_arc (start 146.05 72.39) (end 146.05 71.12) (angle 90) (layer Edge.Cuts) (width 0.15))
   (dimension 43.18 (width 0.3) (layer Dwgs.User)
     (gr_text "43,180 mm" (at 125.73 136.605) (layer Dwgs.User)
